Commit message: - Changes made to ball_chaser CMakeLists to enable proper compiling. - Color added to my_robot.xacro - Updated my_robot wheel dims - Removed ball_chaser.lanuch from world.launch

File: my_robot/urdf/my_robot.xacro (robot description, xacro)
@@ -33,4 +33,7 @@
         </visual>
     </link>
+    <gazebo reference="chassis">
+      <material>Gazebo/Blue</material>
+    </gazebo>
     <link name="front_caster">
       <pose> 0 0 0.08 0 0 0 </pose>
@@ -51,7 +54,4 @@
             <sphere radius="0.08"/>
         </geometry>
-        <material name = "Blue">
-          <color rgba="0.0 0.0 0.5 1.0"/>
-        </material>
         </visual>
     </link>
@@ -82,7 +82,4 @@
             <sphere radius="0.08"/>
         </geometry>
-        <material name = "Blue">
-          <color rgba="0.0 0.0 0.5 1.0"/>
-        </material>
       </visual>
     </link>
@@ -109,5 +106,5 @@
         <origin xyz="0.0 0 0" rpy=" 0 1.5707 1.5707"/>
         <geometry>
-          <cylinder length="0.075" radius="0.155"/>
+          <cylinder length="0.06" radius="0.155"/>
         </geometry>
       </collision>
@@ -117,11 +114,8 @@
           <cylinder length="0.06" radius="0.155"/>
         </geometry>
-        <material name = "Red">
-          <color rgba="0.2 0.2 0.6 1.0"/>
-        </material>
       </visual>
     </link>
     <joint type="continuous" name="left_wheel_hinge">
-        <origin xyz="0 0.13 0" rpy="0 0 0"/>
+        <origin xyz="0 0.135 0" rpy="0 0 0"/>
         <child link="left_wheel"/>
         <parent link="chassis"/>
@@ -150,13 +144,10 @@
       <origin xyz="0.0 0 0" rpy=" 0 1.5707 1.5707"/>
         <geometry>
-          <cylinder length="0.075" radius="0.155"/>
-        </geometry>
-        <material name = "Red">
-          <color rgba="0.2 0.2 0.6 1.0"/>
-        </material>
+          <cylinder length="0.06" radius="0.155"/>
+        </geometry>
       </visual>
     </link>
     <joint type="continuous" name="right_wheel_hinge">
-        <origin xyz="0 -0.13 0" rpy="0 0 0"/>
+        <origin xyz="0 -0.135 0" rpy="0 0 0"/>
         <child link="right_wheel"/>
         <parent link="chassis"/>
@@ -176,7 +167,4 @@
           <box size="0.05 0.05 0.05"/>
         </geometry>
-        <material name = "Red">
-          <color rgba="1.0 0.0 0.0 1.0"/>
-        </material>
       </visual>
       <collision name = "camera_collision">
